Commit message: post beach pond config

File: wamv_rise_description/urdf/base.urdf.xacro (robot description, xacro)
@@ -66,5 +66,5 @@
     <link name="norbit"/>
     <joint name="norbit_joint" type="fixed">
-        <origin xyz="-1.21435 -0.096718 -0.909" rpy="2.094395 0.0 0.0"/>
+        <origin xyz="-1.21435 -0.096718 -0.909" rpy="2.61 0.0 0.0"/>
         <parent link="nose_tip_link"/>
         <child link="norbit"/>

Commit message: add bringup for pi's sensors

File: wamv_rise_description/urdf/base.urdf.xacro (robot description, xacro)
@@ -21,10 +21,16 @@
         <child link="imu"/>
     </joint>
-    <!-- <link name="imu_sf"/>
-    <joint name="imu__sf_joint" type="fixed">
-        <origin xyz="0.0 0.0 0.0" rpy="0.0 0.0 0.0"/>
-        <parent link="imu"/>
-        <child link="imu_sf"/>
-    </joint> -->
+    <link name="gps"/>
+    <joint name="gps_joint" type="fixed">
+        <origin xyz="-0.73 -0.06 0.105" rpy="0.0 0.0 0.0"/>
+        <parent link="base_link"/>
+        <child link="gps"/>
+    </joint>
+    <!-- <link name="rtk_gps"/>
+    <joint name="rtk_gps_joint" type="fixed">
+        <origin xyz="-0.73 -0.06 0.105" rpy="0.0 0.0 0.0"/>
+        <parent link="base_link"/>
+        <child link="gps"/>
+    </joint>     -->
     <!-- <link name="dvl"/>
     <joint name="dvl_joint" type="fixed">
@@ -33,16 +39,4 @@
         <child link="dvl"/>
     </joint> -->
-     <!-- <link name="dvl_sf"/>
-    <joint name="dvl_sf_joint" type="fixed">
-        <origin xyz="0.51 0.0 -0.1" rpy="0.0 0.0 0.0"/>
-        <parent link="base_link"/>
-        <child link="dvl_sf"/>
-    </joint> -->
-    <link name="gps"/>
-    <joint name="gps_joint" type="fixed">
-        <origin xyz="-0.73 -0.06 0.105" rpy="0.0 0.0 0.0"/>
-        <parent link="base_link"/>
-        <child link="gps"/>
-    </joint>
     <!-- <link name="pressure"/>
     <joint name="pressure_joint" type="fixed">
@@ -70,3 +64,16 @@
         <child link="norbit"/>
     </joint>
+    <!-- sf sim sensors -->
+    <!-- <link name="imu_sf"/>
+    <joint name="imu__sf_joint" type="fixed">
+        <origin xyz="0.0 0.0 0.0" rpy="0.0 0.0 0.0"/>
+        <parent link="imu"/>
+        <child link="imu_sf"/>
+    </joint> -->
+     <!-- <link name="dvl_sf"/>
+    <joint name="dvl_sf_joint" type="fixed">
+        <origin xyz="0.51 0.0 -0.1" rpy="0.0 0.0 0.0"/>
+        <parent link="base_link"/>
+        <child link="dvl_sf"/>
+    </joint> -->
 </robot>

Commit message: wamv test update

File: wamv_rise_description/urdf/base.urdf.xacro (robot description, xacro)
@@ -33,10 +33,10 @@
         <child link="gps"/>
     </joint>     -->
-    <!-- <link name="dvl"/>
+    <link name="nortek_dvl"/>
     <joint name="dvl_joint" type="fixed">
-        <origin xyz="0.51 0.0 -0.1" rpy="3.1415926 0.0 0.0"/>
-        <parent link="base_link"/>
-        <child link="dvl"/>
-    </joint> -->
+        <origin xyz="-1.21435 -0.096718 -0.909" rpy="0.0 0.0 0.0"/>
+        <parent link="nose_tip_link"/>
+        <child link="nortek_dvl"/>
+    </joint>
     <!-- <link name="pressure"/>
     <joint name="pressure_joint" type="fixed">

Commit message: added files for mvp

File: wamv_rise_description/urdf/base.urdf.xacro (robot description, xacro)
@@ -77,3 +77,15 @@
         <child link="dvl_sf"/>
     </joint> -->
+    <link name="port_thruster_link"/>
+    <joint name="port_thruster_joint" type="fixed">
+        <origin xyz="-0.77 0.5 -0.1" rpy="0.0 0.0 0.0"/>
+        <parent link="nose_tip_link"/>
+        <child link="port_thruster_link"/>
+    </joint>
+    <link name="starboard_thruster_link"/>
+    <joint name="starboard_thruster_joint" type="fixed">
+        <origin xyz="-0.77 -0.5 -0.1" rpy="0.0 0.0 0.0"/>
+        <parent link="nose_tip_link"/>
+        <child link="starboard_thruster_link"/>
+    </joint>
 </robot>

Commit message: test localization

File: wamv_rise_description/urdf/base.urdf.xacro (robot description, xacro)
@@ -26,4 +26,10 @@
         <parent link="base_link"/>
         <child link="gps"/>
+    </joint>
+    <link name="unicore_gps"/>
+    <joint name="unicore_gps_joint" type="fixed">
+        <origin xyz="0.26 0.0 0.0" rpy="0.0 0.0 0.0"/>
+        <parent link="gps"/>
+        <child link="unicore_gps"/>
     </joint>
     <!-- <link name="rtk_gps"/>
@@ -64,4 +70,10 @@
         <child link="norbit"/>
     </joint>
+    <link name="usbl"/>
+    <joint name="usbl_joint" type="fixed">
+        <origin xyz="-1.21435 -0.096718 -0.909" rpy="0.0 0.0 0.78539815"/>
+        <parent link="nose_tip_link"/>
+        <child link="usbl"/>
+    </joint>
     <!-- sf sim sensors -->
     <!-- <link name="imu_sf"/>

Commit message: change the USBL mounting angle

File: wamv_rise_description/urdf/base.urdf.xacro (robot description, xacro)
@@ -72,5 +72,5 @@
     <link name="usbl"/>
     <joint name="usbl_joint" type="fixed">
-        <origin xyz="-1.21435 -0.096718 -0.909" rpy="0.0 0.0 0.78539815"/>
+        <origin xyz="-1.21435 -0.096718 -0.909" rpy="0.0 0.0 1.221730456"/>
         <parent link="nose_tip_link"/>
         <child link="usbl"/>

Commit message: wamv test including mvp

File: wamv_rise_description/urdf/base.urdf.xacro (robot description, xacro)
@@ -9,10 +9,10 @@
         <child link="nose_tip_link"/>
     </joint>
-    <!-- <link name="cg_link"/>
+    <link name="cg_link"/>
     <joint name="cg_joint" type="fixed">
         <origin xyz="0.0 0.0 0.0" rpy="3.1415926 0.0 0.0"/>
         <parent link="base_link"/>
         <child link="cg_link"/>
-    </joint> -->
+    </joint>
     <link name="imu"/>
     <joint name="imu_joint" type="fixed">
@@ -76,4 +76,16 @@
         <child link="usbl"/>
     </joint>
+    <link name="port_thruster_link"/>
+    <joint name="port_thruster_joint" type="fixed">
+        <origin xyz="-0.77 0.5 -0.1" rpy="0.0 0.0 0.0"/>
+        <parent link="nose_tip_link"/>
+        <child link="port_thruster_link"/>
+    </joint>
+    <link name="starboard_thruster_link"/>
+    <joint name="starboard_thruster_joint" type="fixed">
+        <origin xyz="-0.77 -0.5 -0.1" rpy="0.0 0.0 0.0"/>
+        <parent link="nose_tip_link"/>
+        <child link="starboard_thruster_link"/>
+    </joint>
     <!-- sf sim sensors -->
     <!-- <link name="imu_sf"/>

Commit message: update control and more after salt pond test

File: wamv_rise_description/urdf/base.urdf.xacro (robot description, xacro)
@@ -41,5 +41,6 @@
     <link name="nortek_dvl"/>
     <joint name="dvl_joint" type="fixed">
-        <origin xyz="-1.21435 -0.096718 -0.909" rpy="0.0 0.0 0.0"/>
+        <!-- <origin xyz="-1.21435 -0.096718 -0.909" rpy="0.0 0.0 0.0"/> -->
+        <origin xyz="-1.21435 0.10 -0.909" rpy="0.0 0.0 0.0"/>
         <parent link="nose_tip_link"/>
         <child link="nortek_dvl"/>
@@ -72,5 +73,5 @@
     <link name="usbl"/>
     <joint name="usbl_joint" type="fixed">
-        <origin xyz="-1.21435 -0.096718 -0.909" rpy="0.0 0.0 1.221730456"/>
+        <origin xyz="-1.21435 -0.096718 -0.909" rpy="0.0 0.0 -0.349065844"/>
         <parent link="nose_tip_link"/>
         <child link="usbl"/>

Commit message: update after second prev salt pond mission test

File: wamv_rise_description/urdf/base.urdf.xacro (robot description, xacro)
@@ -41,6 +41,6 @@
     <link name="nortek_dvl"/>
     <joint name="dvl_joint" type="fixed">
-        <!-- <origin xyz="-1.21435 -0.096718 -0.909" rpy="0.0 0.0 0.0"/> -->
-        <origin xyz="-1.21435 0.10 -0.909" rpy="0.0 0.0 0.0"/>
+        <!-- <origin xyz="-1.21435 0.10 -0.909" rpy="0.0 0.0 0.0"/> -->
+        <origin xyz="-1.4352 0.0375 -0.909" rpy="3.1415926 0.0 -1.5707963"/>
         <parent link="nose_tip_link"/>
         <child link="nortek_dvl"/>

Commit message: add power related

File: wamv_rise_description/urdf/base.urdf.xacro (robot description, xacro)
@@ -41,5 +41,4 @@
     <link name="nortek_dvl"/>
     <joint name="dvl_joint" type="fixed">
-        <!-- <origin xyz="-1.21435 0.10 -0.909" rpy="0.0 0.0 0.0"/> -->
         <origin xyz="-1.4352 0.0375 -0.909" rpy="3.1415926 0.0 -1.5707963"/>
         <parent link="nose_tip_link"/>
@@ -73,5 +72,5 @@
     <link name="usbl"/>
     <joint name="usbl_joint" type="fixed">
-        <origin xyz="-1.21435 -0.096718 -0.909" rpy="0.0 0.0 -0.349065844"/>
+        <origin xyz="-1.21435 -0.096718 -1.0" rpy="0.0 0.0 -0.349065844"/>
         <parent link="nose_tip_link"/>
         <child link="usbl"/>
