Commit message: set all the bringup for pi4

File: wamv_rise_description/urdf/base.urdf (robot description, URDF)
Before this commit: robot wamv_rise, 10 links, 9 joints
Links:
- added link cg_link
- added link unicore_gps
- added link usbl
Joints:
- added joint cg_joint: type fixed, parent base_link, child cg_link, origin xyz=0.0 0.0 0.0 rpy=3.1415926 0.0 0.0
- added joint unicore_gps_joint: type fixed, parent gps, child unicore_gps, origin xyz=0.26 0.0 0.0 rpy=0.0 0.0 0.0
- added joint usbl_joint: type fixed, parent nose_tip_link, child usbl, origin xyz=-1.21435 -0.096718 -1.0 rpy=0.0 0.0 -0.349065844
- joint dvl_joint: origin xyz=-1.21435 -0.096718 -0.909 rpy=0.0 0.0 0.0 -> xyz=-1.4352 0.0375 -0.909 rpy=3.1415926 0.0 -1.5707963

Commit message: added simulation files

File: wamv_rise_description/urdf/base.urdf (robot description, URDF)
Before this commit: robot wamv_rise, 13 links, 12 joints
Links:
- added link dvl_sf
- added link imu_sf
Joints:
- added joint dvl_sf_joint: type fixed, parent nose_tip_link, child dvl_sf, origin xyz=-1.4352 0.0375 -0.909 rpy=0.0 0.0 0.0
- added joint imu_sf_joint: type fixed, parent base_link, child imu_sf, origin xyz=0.0 0.0 0.0 rpy=0.0 0.0 0.0

Commit message: add usb gps && fix urdf

File: wamv_rise_description/urdf/base.urdf (robot description, URDF)
Before this commit: robot wamv_rise, 15 links, 14 joints
Links:
- removed link gps
- added link usb_gps
Joints:
- removed joint gps_joint
- added joint usb_gps_joint: type fixed, parent nose_tip_link, child usb_gps, origin xyz=-1.0 0.0 0.0 rpy=0.0 0.0 0.0
- joint imu_joint: origin xyz=0.0 0.0 0.0 rpy=0.0 0.0 3.1415926 -> xyz=0.0 0.06 0.0 rpy=0.0 0.0 3.1415926
- joint nose_tip_joint: origin xyz=1.11 -0.06 0.16 rpy=0.0 0.0 0.0 -> xyz=1.11 0.0 0.16 rpy=0.0 0.0 0.0
- joint port_thruster_joint: parent nose_tip_link -> base_link
- joint starboard_thruster_joint: parent nose_tip_link -> base_link
- joint unicore_gps_joint: origin xyz=0.26 0.0 0.0 rpy=0.0 0.0 0.0 -> xyz=-0.47 0.0 0.105 rpy=0.0 0.0 0.0; parent gps -> base_link

Commit message: new microstrain imu and c2 traffic manager

File: wamv_rise_description/urdf/base.urdf (robot description, URDF)
Before this commit: robot wamv_rise, 15 links, 14 joints
Joints:
- joint imu_joint: origin xyz=0.0 0.06 0.0 rpy=0.0 0.0 3.1415926 -> xyz=0.15 -0.06 0.05 rpy=0.0 0.0 0.0
