Commit message: feat: link for dvl pressure

File: wamv_rise_description/urdf/base.urdf (robot description, URDF)
Before this commit: robot wamv_rise, 15 links, 14 joints
Links:
- added link nortek_dvl_pressure
Joints:
- added joint dvl_joint_pressure: type fixed, parent nose_tip_link, child nortek_dvl_pressure, origin xyz=-1.4352 0.0375 -0.909 rpy=0.0 0.0 -1.5707963

Commit message: fix#2 & child frame for depth odometry

File: wamv_rise_description/urdf/base.urdf (robot description, URDF)
Before this commit: robot wamv_rise, 16 links, 15 joints
Links:
- added link airmar_link
Joints:
- added joint airmar_joint: type fixed, parent nose_tip_link, child airmar_link, origin xyz=-1.4352 0.16 1.0 rpy=0.0 0.0 0.0
